File: pcb/anemo.kicad_pcb (KiCad board)
At the start: 2 copper layers, 47 x 53 mm, 21 parts, among them J1 Screw_Terminal_01x02, J2 Screw_Terminal_01x02, U1 LM393, U2 ESP32_DEVCITV1

Commit message: pcb to kicad10 format
Parts:
- moved C3 0.79 mm to (88.3, 101.0)
Routing:
- net VCC: track 84.3 -> 83.5 mm

Commit message: v1.0 gerber
Other:
- board text added: "Anemo v1.0"
